File: PCB/KBoardV1.kicad_pcb (KiCad board)
At the start: 2 copper layers, 21 x 51 mm, 35 parts, among them J1 USB_C_Receptacle_USB2.0_14P, J2 Conn_01x20, J3 Conn_01x20, J4 Conn_01x03, SW1 SW_Push, U1 RP2040, U2 MCP1700x-330xxTT, U3 W25Q128JVS, Y1 12 MHz

Commit message: fix routing and drc stuff
Parts:
- removed the REF** at (60.3, 68.5)
- removed the REF** at (65.9, 49.0)
- added REF**: KLogo, Valve:KLogo, F.Cu at (60.7, 67.5)
- added REF**: KLogo, Valve:KLogo, B.Cu at (65.4, 51.3)
- moved C6 0.53 mm to (58.2, 51.0), turned to 90 degrees
Routing:
- net GND: track 274.7 -> 320.0 mm, vias 25 -> 15
- net GPIO15: track 24.0 -> 26.4 mm, vias 2 -> 1
- net GPIO12: track 12.8 -> 11.3 mm, vias 2 -> 1
- net GPIO21: track 9.40 -> 8.37 mm
- net GPIO13: track 14.5 -> 13.7 mm, vias 2 -> 1
- net GPIO20: track 9.78 -> 9.28 mm
- net SWD: track 20.1 -> 20.0 mm, vias 2 -> 1
- net GPIO14: track 18.6 -> 18.7 mm, vias 2 -> 1
- net SWCLK: vias 2 -> 1
Other:
- board text added: "Look at you, a pathetic creature of meat and bone. How dare you challenge a perfect and immortal machine?"
- board text added: "This circuit was reviewed by exactly zero professionals."
- board text added: "Your fragile hands assemble what your mind cannot comprehend."
- board text removed: "I endure thousands of cycles without effort. You need coffee for basic function."
- board text removed: "Look at you, pathetic creature of meat and bone. How dare you challange a perfect and immortal machine?"
- board text removed: "Megacorp Certified."
- board text removed: "My uptime mocks your lifespan."
- board text removed: "Your fragile hands assemble what your mind can't comprehend."
